File: doc/designspec/schematics/brain/brain.sch (KiCad schematic (older format))
At the start: 7 parts, among them P1 USB_RPi_2, P2 USB_RPi_1, P3 RPi_3_GPIO

Commit message: Add reset signal to brain
Connections:
- net RESET: now reaches P3.7 (P7)
- no-connect marks 36 -> 35
Changed lines of the file:
@@
 NoConn ~ 2750 1550
 NoConn ~ 2750 1450
-NoConn ~ 2750 1350
 NoConn ~ 2750 1250
 NoConn ~ 2750 1150
@@
 Wire Wire Line
 	3350 3000 3550 3000
+Text GLabel 2600 1350 0    60   Input ~ 0
+RESET
+Wire Wire Line
+	2600 1350 2750 1350
 $EndSCHEMATC
