File: doc/designspec/schematics/styrenhet/styrenhet.sch (KiCad schematic (older format))
At the start: 8 parts, among them IC1 ATMEGA1284P-P, U1 IQEXO-3, U2 Terminator-CTRL, U3 USB-UART

Commit message: Fix uart connection in kicad
Connections:
- net at IC1.14 ((PCINT24/RXD0)PD0): now also U3.2 (TX); no longer U3.1 (RX)
- net at IC1.15 ((PCINT25/TXD0)PD1): now also U3.1 (RX); no longer U3.2 (TX)
Other:
- moved on the sheet: U3
Changed lines of the file:
@@
 L USB-UART U3
 U 1 1 57F7998E
-P 6350 4750
-F 0 "U3" H 6000 4900 60  0000 C CNN
-F 1 "USB-UART" H 6350 4750 60  0000 C CNN
-F 2 "" H 6350 4750 60  0001 C CNN
-F 3 "" H 6350 4750 60  0001 C CNN
-	1    6350 4750
+P 6550 4750
+F 0 "U3" H 6200 4900 60  0000 C CNN
+F 1 "USB-UART" H 6550 4750 60  0000 C CNN
+F 2 "" H 6550 4750 60  0001 C CNN
+F 3 "" H 6550 4750 60  0001 C CNN
+	1    6550 4750
 	1    0    0    -1
 $EndComp
@@
 	1    0    0    -1
 $EndComp
+Wire Wire Line
+	5950 4700 5900 4700
+Wire Wire Line
+	5900 4700 5900 4750
+Wire Wire Line
+	5900 4750 5800 4750
+Wire Wire Line
+	5800 4750 5800 4800
+Wire Wire Line
+	5800 4800 5750 4800
+Wire Wire Line
+	5750 4700 5850 4700
+Wire Wire Line
+	5850 4700 5850 4800
+Wire Wire Line
+	5850 4800 5950 4800
 $EndSCHEMATC
